File: msisdr.kicad_sch (KiCad schematic)
At the start: 0 parts

Commit message: initial schematic work done on v2
Parts:
- added C1, C22, C3, C30, C38, C4, C47: 10nF, symbol Device:C_Small
- added C10, C21, C37, C39, C41, C42, C44, C45, C48, C50, C51: 1uF, symbol Device:C_Small
- added C11: 200pF, symbol Device:C_Small
- added C12: 68pF, symbol Device:C_Small
- added C13, C16, C19, C20, C40, C49, C6, C9: 0.1uF, symbol Device:C_Small
- added C14: 24pF, symbol Device:C_Small
- added C15: 150pF, symbol Device:C_Small
- added C17: 56pF, symbol Device:C_Small
- added C18, C29: 10uF, symbol Device:C_Polarized_Small
- added C2: 82pF, symbol Device:C_Small
- added C23: 6.8nF, symbol Device:C_Small
- added C24: 22pF, symbol Device:C_Small
- added C25: 3.9pF, symbol Device:C_Small
- added C26: 33nF, symbol Device:C_Small
- added C27: 8.2pF, symbol Device:C_Small
- added C28: 3.6pF, symbol Device:C_Small
- added C31: 51pF, symbol Device:C_Small
- added C32: 9.1pF, symbol Device:C_Small
- added C33, C36: 6.8pF, symbol Device:C_Small
- added C34: 3pF, symbol Device:C_Small
- added C35: 39pF, symbol Device:C_Small
- added C43: 2.4pF, symbol Device:C_Small
- added C46: 2pF, symbol Device:C_Small
- added C5, C8: 30pF, symbol Device:C_Small
- added C7: 180pF, symbol Device:C_Small
- added D1: PWR, symbol Device:LED_Small
- added FB1: 10uH, symbol Device:FerriteBead_Small
- added J1: HF, symbol Connector:Conn_Coaxial
- added J2: VHF+, symbol Connector:Conn_Coaxial
- added J3: USB_B_Micro, symbol Connector:USB_B_Micro
- added J4: GPIO, symbol Connector:Conn_01x06_Female
- added L1, L4: 130nH, symbol Device:L_Small
- added L10, L13: 16nH, symbol Device:L_Small
- added L11: 100nH, symbol Device:L_Small
- added L12: 18nH, symbol Device:L_Small
- added L14: 6.8nH, symbol Device:L_Small
- added L15: 120nH, symbol Device:L_Small
- added L16: 22nH, symbol Device:L_Small
- added L17: 20nH, symbol Device:L_Small
- added L18: 9.1nH, symbol Device:L_Small
- added L19: 11nH, symbol Device:L_Small
- added L2: 360nH, symbol Device:L_Small
- added L20: 4.7nH, symbol Device:L_Small
- added L21: 6.2nH, symbol Device:L_Small
- added L3, L6: 470nH, symbol Device:L_Small
- added L5: 56nH, symbol Device:L_Small
- added L7: 160nH, symbol Device:L_Small
- added L8: 75nH, symbol Device:L_Small
- added L9: 39nH, symbol Device:L_Small
- added R1, R2: 22R, symbol Device:R_Small
- added R3: 390, symbol Device:R_Small
- added R4, R5: 510, symbol Device:R_Small
- added U1: MSI001, Housings_DFN_QFN:QFN-40-1EP_6x6mm_Pitch0.5mm, symbol msi001:msi001
- added U2: LP5907MFX-3.3, Package_TO_SOT_SMD:SOT-23-5, symbol Regulator_Linear:LP5907MFX-3.3
- added U3: LP5907MFX-2.8, Package_TO_SOT_SMD:SOT-23-5, symbol Regulator_Linear:LP5907MFX-2.8
- added U4: MSI2500, Housings_DFN_QFN:QFN-32-1EP_5x5mm_Pitch0.5mm, symbol msi:msi2500
- added Y1: 24.0000 MHz, symbol Device:Crystal_GND24_Small
Connections:
- new net: C43.2, C46.1, L20.2
- new net: FB1.1, J3.1 (VBUS)
- new net: C10.1, C21.1, FB1.2, U2.1 (IN), U2.3 (EN), U3.1 (IN)
- new net: C8.2, L4.1
- new net: C12.1, C14.1, L4.2, L5.2
- new net: C45.1, U4.16 (V18_PHY)
- new net: D1.2 (A), R5.2
- new net: C13.1, U1.39 (INB)
- new net: C2.1, J1.1 (In), L2.1
- new net: C7.1, L2.2, L3.1
- new net: C31.1, C33.1, L11.2, L13.2
- new net: C4.1, U1.9 (INB)
- new net: C39.2, U4.13 (V18_ADC)
- new net: C48.1, U4.17 (V15_VCO)
- new net: R4.2, U4.21 (REST)
- new net: C51.1, U4.22 (X0), Y1.3
- new net: C50.1, U4.23 (X1), Y1.1
- new net: C47.1, U4.24 (REFOUT)
- new net: C38.2, U4.6 (ADC_REF_P)
- new net: C38.1, U4.7 (ADC_REF_N)
- new net: C11.1, L3.2, L6.1
- new net: C23.2, C30.2, R3.1, U1.28 (VCO-VCC)
- new net: C26.2, R3.2, U1.26 (LFILT-PC)
- new net: J3.3 (D+), R1.1
- new net: J3.2 (D-), R2.2
- new net: C32.1, C34.1, L12.2, L14.2
- new net: C28.2, L12.1
- new net: C1.1, U1.7 (INB)
- new net: C23.1, C26.1, U1.27 (CP-OUT)
- new net: C34.2, L16.1
- new net: C22.2, U1.25 (INB)
- new net: C33.2, L15.1
- new net: C9.2, U1.40 (IN)
- new net: C3.1, U1.4 (INB)
- new net: C27.2, L11.1
- new net: C14.2, L7.1
- new net +1V8: C41.1, U4.31 (V18_DIGITAL)
- new net +2V8: C16.1, C19.1, C20.1, C29.1, C6.1, U1.1 (VCC1), U1.14 (VCC5), U1.15 (VCC6), U1.18 (VCC7), U1.19 (VCC8), U1.2 (VCC2), U1.23 (VCC9), U1.29 (VCC10), U1.30 (VCC11), U1.31 (VDDI), U1.32 (VDD), U1.36 (VCC12), U1.8 (VCC3), U3.5 (OUT)
- new net +3V3: C18.1, C40.2, C42.2, C49.1, R5.1, U2.5 (OUT), U4.14 (VCC_3V_PM), U4.18 (VCC_3V_XCVR), U4.32 (VCC_3V_DIGITAL)
- new net GND: C1.2, C10.2, C11.2, C12.2, C13.2, C15.2, C16.2, C17.2, C18.2, C19.2, C2.2, C20.2, C21.2, C22.1, C24.2, C25.2, C29.2, C3.2, C30.1, C31.2, C32.2, C35.2, C36.2, C37.1, C39.1, C4.2, C40.1, C41.2, C42.1, C44.2, C45.2, C48.2, C49.2, C5.2, C50.2, C51.2, C6.2, C7.2, D1.1 (K), J1.2 (Ext), J2.2 (Ext), J3.5 (GND), J3.6 (Shield), J4.6 (Pin_6), L1.1, L10.1, L13.1, L14.1, L17.1, L18.1, L19.1, L20.1, L21.1, L5.1, L8.1, L9.1, R4.1, U1.41 (GND), U2.2 (GND), U3.2 (GND), U4.28 (XTAL_SEL), U4.29 (TEST1), U4.30 (TEST2), U4.33 (GND), U4.8 (VEE_ADC), Y1.2, Y1.4
- new net GPIO0: J4.2 (Pin_2), U4.2 (GPIO_0)
- new net GPIO1: J4.3 (Pin_3), U4.3 (GPIO_1)
- new net GPIO2: J4.4 (Pin_4), U4.4 (GPIO_2)
- new net GPIO3: J4.5 (Pin_5), U4.5 (GPIO_3)
- new net HF: C15.1, C9.1, L6.2
- new net I+: U1.11 (OPI), U4.9 (IIN_P)
- new net I-: U1.12 (OPIB), U4.10 (IIN_N)
- new net Q+: U1.22 (OPQ), U4.11 (QIN_P)
- new net Q-: U1.21 (OPQB), U4.12 (QIN_N)
- new net REFCLK: C47.2, U1.20 (REF-CLK)
- new net SPI_CLK: U1.34 (CLK), U4.27 (SPI_CLK)
- new net SPI_DATA: U1.35 (DATA), U4.26 (SPI_DAT)
- new net SPI_LAT: U1.33 (EN), U4.25 (SPI_LAT)
- new net UHF_H: C46.2, L21.2, U1.24 (IN)
- new net UHF_L: C36.1, L16.2, L18.2, U1.6 (IN)
- new net USB_DM: R2.1, U4.20 (DM)
- new net USB_DP: R1.2, U4.19 (DP)
- new net V18_SYNTH: C44.1, U3.3 (EN), U4.15 (V18_SYNTH)
- new net VHF+: C24.1, C25.1, C27.1, C28.1, C43.1, C5.1, C8.1, J2.1 (In), L1.2, L10.2, L19.2, L9.2
- new net VHF_H: C35.1, L15.2, L17.2, U1.3 (IN)
- new net VHF_L: C17.1, L7.2, L8.2, U1.10 (IN)
- new net V_GPIO: C37.2, J4.1 (Pin_1), U4.1 (VCC_GPIO)
- no-connect marks 0 -> 7
Other:
- removed sheet MSI2500
- removed sheet msi001
- removed sheet power&interface
- removed sheet rf_parts
- note added: "(50Ω input, 100Ω output)"
- note added: "1000MHz Chebyshev HPF"
- note added: "130-240MHz Chebyshev BPF"
- note added: "2.8V Supply disabled until MSI2500 internal regulators ready"
- note added: "30MHz Chebyshev LPF"
- note added: "400-1000MHz Chebyshev BPF"
- note added: "50-130MHz Chebyshev BPF"
- company: (none) -> W3AXL
- title: (none) -> msiSDRv2
